Commit message: Working writing but not reading

File: xarm_description/urdf/xarm.urdf (robot description, URDF)
Before this commit: robot xarm, 6 links, 5 joints
Links:
- added link xarm_1_link, mass 0.1; collision box size=0.1 0.1 0.1; visual box size=0.1 0.1 0.1
Joints:
- added joint xarm_1_joint: type revolute, parent xarm_2_link, child xarm_1_link, origin xyz=0 -0.001205 0.05306 rpy=0 0 0, axis 0 0 1, limit lower=0.0 upper=1.0 effort=1000 velocity=1.0

Commit message: urdf of gripper ready

File: xarm_description/urdf/xarm.urdf (robot description, URDF)
Before this commit: robot xarm, 7 links, 6 joints
Links:
- link xarm_1_link: geometry collision mesh filename=package://xarm_description/meshes/stls/gripper.stl scale=1.0 1.0 1.0; visual mesh filename=package://xarm_description/meshes/stls/gripper.stl scale=1.0 1.0 1.0
Joints:
- joint xarm_1_joint: origin xyz=0 -0.001205 0.05306 rpy=0 0 0 -> xyz=0 0 0.007548 rpy=0 0 0

Commit message: Added gripper_tip link

File: xarm_description/urdf/xarm.urdf (robot description, URDF)
Before this commit: robot xarm, 7 links, 6 joints
Links:
- added link xarm_gripper_tip
Joints:
- added joint xarm_gripper_tip_joint: type fixed, parent xarm_2_link, child xarm_gripper_tip, origin xyz=0.0 0.0 0.104639 rpy=0.0 0.0 0.0
